File: grbl-db25.kicad_pcb (KiCad board)
At the start: 2 copper layers, 4 parts, among them J1 Conn_02x03_Odd_Even, J2 Conn_02x01, J3 DB25_Male

Commit message: one side soldering
Parts:
- moved J2 5.08 mm to (110.5, 123.2)
- moved J1 2.54 mm to (110.5, 133.3)
Connections:
- D1 pad 10: IN3Y -> IN2X
- D1 pad 11: PWM -> IN3Y
- D1 pad 9: IN2X -> PWM
- D1 pad A0: STOP -> RELAY2MIST
- D1 pad A1: HOLD -> STOP
- D1 pad A2: START -> HOLD
- D1 pad A3: RELAY2MIST -> START
Routing:
- net IN1-ESTOP: track 0.00 -> 25.7 mm, vias 0 -> 1
- net GND: track 28.8 -> 52.3 mm, vias 0 -> 1
- net ENABLE: track 0.00 -> 21.8 mm, vias 0 -> 1
- net PWM: track 0.00 -> 17.1 mm
- net STEP1X: track 41.3 -> 57.8 mm, vias 0 -> 1
- net STEP2Y: track 37.1 -> 51.0 mm, vias 0 -> 1
- net IN2X: track 27.7 -> 15.4 mm, vias 2 -> 1
- net STEP3Z: track 32.8 -> 44.3 mm, vias 0 -> 1
- net IN3Y: track 16.6 -> 19.8 mm, vias 0 -> 1
- net RELAY2MIST: track 46.6 -> 43.6 mm
- net DIR3Z: track 28.7 -> 30.7 mm, vias 0 -> 1
- net DIR2Y: track 25.0 -> 26.2 mm, vias 0 -> 1
- net DIR1X: track 23.8 -> 24.7 mm, vias 0 -> 1
- net IN4Z: track 23.4 -> 23.7 mm, vias 0 -> 1
- added copper zone on B.Cu, net GND
- added copper zone on F.Cu, net GND
Other:
- board outline added: 38.1 x 80 mm
- net class Default: via_dia 1.2 -> 1.5; via_drill 0.4 -> 0.6
