File: grbl-db25.sch (KiCad schematic (older format))
At the start: 4 parts, among them J1 Conn_02x03_Odd_Even, J2 Conn_02x01, J3 DB25_Male

Commit message: one side soldering
Connections:
- net HOLD: now also D1.A2; no longer D1.A1
- net IN2X: now also D1.10; no longer D1.9
- net IN3Y: now also D1.11; no longer D1.10
- net PWM: now also D1.9; no longer D1.11
- net RELAY2MIST: now also D1.A0; no longer D1.A3
- net START: now also D1.A3; no longer D1.A2
- net STOP: now also D1.A1; no longer D1.A0
Changed lines of the file:
@@
 Text GLabel 3250 3750 0    50   Output ~ 0
 ENABLE
-Text GLabel 4700 3950 2    50   Output ~ 0
+Text GLabel 3250 3850 0    50   Output ~ 0
 PWM
-Text GLabel 4700 3650 2    50   Input ~ 0
+Text GLabel 4700 3550 2    50   Input ~ 0
 STOP
-Text GLabel 4700 3550 2    50   Input ~ 0
+Text GLabel 4700 3450 2    50   Input ~ 0
 HOLD
-Text GLabel 4700 3450 2    50   Input ~ 0
+Text GLabel 4700 3250 2    50   Input ~ 0
 START
 Text GLabel 5350 1900 2    50   Input ~ 0
@@
 Text GLabel 4700 3350 2    50   Output ~ 0
 RELAY1FLOOD
-Text GLabel 4700 3250 2    50   Output ~ 0
+Text GLabel 4700 3650 2    50   Output ~ 0
 RELAY2MIST
-Text GLabel 3250 3850 0    50   Input ~ 0
+Text GLabel 4700 4050 2    50   Input ~ 0
 IN2X
-Text GLabel 4700 4050 2    50   Input ~ 0
+Text GLabel 4700 3950 2    50   Input ~ 0
 IN3Y
 Text GLabel 4700 3850 2    50   Input ~ 0
